File: Amigo.kicad_pcb (KiCad board)
At the start: 2 copper layers, 75.5 x 75 mm, 39 parts, among them J1 USB_C_Receptacle_USB2.0_16P, J2 Conn_01x02, J3 SH1106 OLED, J4 MAX98357A, J5 DRV8833, J6 ButtonRibbonConnector, SW1 SW_Push, SW2 SW_Push, U1 TP4056-42-ESOP8, U2 AP2112K-3.3, U3 ESP32-S3-WROOM-1

Commit message: Found out why there is a discrepancy with two main board files. The real one is in the Main Board folder
Parts:
- removed C1, C11, C2, C3: 10µF, Capacitor_SMD:C_0603_1608Metric
- removed C10, C12, C4, C6, C9: 100nF, Capacitor_SMD:C_0603_1608Metric
- removed C13: 10µF, Capacitor_SMD:C_0805_2012Metric
- removed C5, C7, C8: 1µF, Capacitor_SMD:C_0603_1608Metric
- removed D1, D2, D3: LED, LED_SMD:LED_0805_2012Metric
- removed J1: USB_C_Receptacle_USB2.0_16P, Connector_USB:USB_C_Receptacle_GCT_USB4085
- removed J2: Conn_01x02, Connector_JST:JST_PH_S2B-PH-K_1x02_P2.00mm_Horizontal
- removed J3: SH1106 OLED, Connector_PinHeader_2.54mm:PinHeader_1x04_P2.54mm_Vertical
- removed J4: MAX98357A, Connector_PinHeader_2.54mm:PinHeader_1x07_P2.54mm_Vertical
- removed J5: DRV8833, Connector_PinHeader_2.54mm:PinHeader_1x08_P2.54mm_Vertical
- removed J6: ButtonRibbonConnector, Connector_PinHeader_2.54mm:PinHeader_1x08_P2.54mm_Vertical
- removed R1, R2: 5.1k, Resistor_SMD:R_0603_1608Metric
- removed R10, R11, R12: 1k, Resistor_SMD:R_0603_1608Metric
- removed R3: 2k, Resistor_SMD:R_0603_1608Metric
- removed R4, R5: 100k, Resistor_SMD:R_0603_1608Metric
- removed R6, R7: 10k, Resistor_SMD:R_0603_1608Metric
- removed R8, R9: 4.7k, Resistor_SMD:R_0603_1608Metric
- removed SW1, SW2: SW_Push, Button_Switch_SMD:SW_SPST_TL3342
- removed U1: TP4056-42-ESOP8, Package_SO:SOIC-8-1EP_3.9x4.9mm_P1.27mm_EP2.41x3.3mm_ThermalVias
- removed U2: AP2112K-3.3, Package_TO_SOT_SMD:SOT-23-5
- removed U3: ESP32-S3-WROOM-1, RF_Module:ESP32-S3-WROOM-1
Other:
- board outline removed
