File: ButtonMatrix3x3/ButtonMatrix3x3.kicad_pcb (KiCad board)
At the start: 2 copper layers, 65 x 65 mm, 22 parts, among them J1 ButtonRibbonConnector

Commit message: Main PCB placement
Parts:
- added REF**: MountingHole_3.2mm_M3, MountingHole:MountingHole_3.2mm_M3, F.Cu at (73.5, 15.5)
- added REF**: MountingHole_3.2mm_M3, MountingHole:MountingHole_3.2mm_M3, F.Cu at (15.5, 73.5)
- added REF**: MountingHole_3.2mm_M3, MountingHole:MountingHole_3.2mm_M3, F.Cu at (15.5, 15.5)
- added REF**: MountingHole_3.2mm_M3, MountingHole:MountingHole_3.2mm_M3, F.Cu at (73.5, 73.5)
Routing:
- net (no net): track 0.00 -> 4.91 mm

Commit message: Gerbers generated
Routing:
- net (no net): track 4.91 -> 0.00 mm
Other:
- board text added: ":)"
Changed lines of the file:
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@@
 			(plot_on_all_layers_selection 0x00000000_00000000_00000000_00000000)
 			(disableapertmacros no)
-			(usegerberextensions no)
+			(usegerberextensions yes)
 			(usegerberattributes yes)
 			(usegerberadvancedattributes yes)
@@
 			(sketchdnponfab yes)
 			(crossoutdnponfab yes)
-			(subtractmaskfromsilk no)
+			(subtractmaskfromsilk yes)
 			(outputformat 1)
 			(mirror no)
-			(drillshape 1)
+			(drillshape 0)
 			(scaleselection 1)
-			(outputdirectory "")
+			(outputdirectory "Gerbers/")
 		)
 	)
@@
 		(layer "Edge.Cuts")
 	)
-	(segment
-		(start 22.5 73.5)
-		(end 23 74)
-		(width 0.2)
-		(layer "F.Cu")
-		(net "")
-	)
-	(segment
-		(start 23.5 73.5)
-		(end 23.5 73)
-		(width 0.2)
+	(gr_text ":)"
+		(at 23.5 74 0)
 		(layer "F.Cu")
-		(net "")
-	)
-	(segment
-		(start 25 73.5)
-		(end 25 73)
-		(width 0.2)
-		(layer "F.Cu")
-		(net "")
-	)
-	(segment
-		(start 25.5 74)
-		(end 26 73.5)
-		(width 0.2)
-		(layer "F.Cu")
-		(net "")
-	)
-	(segment
-		(start 23 74)
-		(end 25.5 74)
-		(width 0.2)
-		(layer "F.Cu")
-		(net "")
+		(effects
+			(font
+				(size 1.5 1.5)
+				(thickness 0.3)
+				(bold yes)
+			)
+			(justify left bottom)
+		)
 	)
 	(segment

Commit message: idk tbh
Parts:
- moved R1 7.00 mm to (48.0, 67.0)
- moved R2 7.00 mm to (52.0, 67.0)
- moved R3 7.00 mm to (56.0, 67.0)
- moved REF** 5.00 mm to (15.5, 68.5)
- moved REF** 5.00 mm to (73.5, 68.5)
- moved J1 0.50 mm to (44.5, 69.5)
Routing:
- net BUTTON_ROW_0: track 110.4 -> 79.2 mm
- net BUTTON_ROW_1: track 89.5 -> 63.3 mm
- net BUTTON_COL_2: track 58.0 -> 51.3 mm, vias 0 -> 4
- net BUTTON_COL_1: track 74.8 -> 71.1 mm, vias 0 -> 4
- net BUTTON_ROW_2: track 41.8 -> 44.2 mm
- net +3V3: track 14.4 -> 13.3 mm, vias 0 -> 4
- net BUTTON_COL_0: track 84.6 -> 84.5 mm, vias 2 -> 0
Other:
- board size 65 x 65 mm -> 65 x 60 mm
