File: Amigo Main Board/Amigo.kicad_pcb (KiCad board)
At the start: 2 copper layers, 50 x 50 mm, 39 parts, among them J1 USB_C_Receptacle_USB2.0_16P, J2 Conn_01x02, J3 OLED, J4 MAX98357A, J5 Rocker Switch, J6 ButtonRibbonConnector, SW1 SW_Push, SW2 SW_Push, U1 TP4056-42-ESOP8, U2 AP2112K-3.3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

Commit message: Debugged an unconnected error and generated step and gerber
Routing:
- net GND: vias 2 -> 3
- net (no net): vias 0 -> 1
Changed lines of the file:
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@@
 		)
+	)
+	(via
+		(at 31.25 45.5)
+		(size 0.6)
+		(drill 0.3)
+		(layers "F.Cu" "B.Cu")
+		(net "")
 	)
 	(segment
@@
 	(via
 		(at 40 15.5)
+		(size 0.6)
+		(drill 0.3)
+		(layers "F.Cu" "B.Cu")
+		(net "GND")
+	)
+	(via
+		(at 46.5 20.25)
 		(size 0.6)
 		(drill 0.3)
@@
 	)
 	(segment
+		(start 42 37.825)
+		(end 42 39.5)
+		(width 0.25)
+		(layer "F.Cu")
+		(net "Net-(C10-Pad1)")
+	)
+	(segment
 		(start 22.995 15.495)
 		(end 20.378984 15.495)
@@
 	)
 	(segment
+		(start 36.883884 51.5)
+		(end 34.758884 49.375)
+		(width 0.25)
+		(layer "F.Cu")
+		(net "AUDIO_LRC_WS")
+	)
+	(segment
+		(start 20.83 49.375)
+		(end 20.205 48.75)
+		(width 0.25)
+		(layer "F.Cu")
+		(net "AUDIO_LRC_WS")
+	)
+	(segment
+		(start 19.670603 46.420603)
+		(end 19.670603 45.568961)
+		(width 0.25)
+		(layer "F.Cu")
+		(net "AUDIO_LRC_WS")
+	)
+	(segment
+		(start 34.758884 49.375)
+		(end 27.458883 49.375)
+		(width 0.25)
+		(layer "F.Cu")
+		(net "AUDIO_LRC_WS")
+	)
+	(segment
+		(start 20.205 46.955)
+		(end 19.670603 46.420603)
+		(width 0.25)
+		(layer "F.Cu")
+		(net "AUDIO_LRC_WS")
+	)
+	(segment
+		(start 20.205 48.75)
+		(end 20.205 46.955)
+		(width 0.25)
+		(layer "F.Cu")
+		(net "AUDIO_LRC_WS")
+	)
+	(segment
+		(start 44.5 51.5)
+		(end 36.883884 51.5)
+		(width 0.25)
+		(layer "F.Cu")
+		(net "AUDIO_LRC_WS")
+	)
+	(via
+		(at 27.458883 49.375)
+		(size 0.6)
+		(drill 0.3)
+		(layers "F.Cu" "B.Cu")
+		(net "AUDIO_LRC_WS")
+	)
+	(via
+		(at 20.83 49.375)
+		(size 0.6)
+		(drill 0.3)
+		(layers "F.Cu" "B.Cu")
+		(net "AUDIO_LRC_WS")
+	)
+	(segment
+		(start 27.458883 49.375)
+		(end 20.83 49.375)
+		(width 0.25)
+		(layer "B.Cu")
+		(net "AUDIO_LRC_WS")
+	)
+	(segment
 		(start 19.251642 47)
 		(end 19.25 47)
@@
 	)
 	(segment
-		(start 36.883884 51.5)
-		(end 34.758884 49.375)
-		(width 0.25)
-		(layer "F.Cu")
-		(net "AUDIO_LRC_WS")
-	)
-	(segment
-		(start 20.83 49.375)
-		(end 20.205 48.75)
-		(width 0.25)
-		(layer "F.Cu")
-		(net "AUDIO_LRC_WS")
-	)
-	(segment
-		(start 19.670603 46.420603)
-		(end 19.670603 45.568961)
-		(width 0.25)
-		(layer "F.Cu")
-		(net "AUDIO_LRC_WS")
-	)
-	(segment
-		(start 34.758884 49.375)
-		(end 27.458883 49.375)
-		(width 0.25)
-		(layer "F.Cu")
-		(net "AUDIO_LRC_WS")
-	)
-	(segment
-		(start 20.205 46.955)
-		(end 19.670603 46.420603)
-		(width 0.25)
-		(layer "F.Cu")
-		(net "AUDIO_LRC_WS")
-	)
-	(segment
-		(start 20.205 48.75)
-		(end 20.205 46.955)
-		(width 0.25)
-		(layer "F.Cu")
-		(net "AUDIO_LRC_WS")
-	)
-	(segment
-		(start 44.5 51.5)
-		(end 36.883884 51.5)
-		(width 0.25)
-		(layer "F.Cu")
-		(net "AUDIO_LRC_WS")
-	)
-	(via
-		(at 27.458883 49.375)
-		(size 0.6)
-		(drill 0.3)
-		(layers "F.Cu" "B.Cu")
-		(net "AUDIO_LRC_WS")
-	)
-	(via
-		(at 20.83 49.375)
-		(size 0.6)
-		(drill 0.3)
-		(layers "F.Cu" "B.Cu")
-		(net "AUDIO_LRC_WS")
-	)
-	(segment
-		(start 27.458883 49.375)
-		(end 20.83 49.375)
-		(width 0.25)
-		(layer "B.Cu")
-		(net "AUDIO_LRC_WS")
-	)
-	(segment
 		(start 44.105 46.025)
 		(end 44.5 46.42)
@@
 		(net "AUDIO_DOUT")
 	)
-	(segment
-		(start 42 37.825)
-		(end 42 39.5)
-		(width 0.25)
-		(layer "F.Cu")
-		(net "Net-(C10-Pad1)")
-	)
 	(zone

Commit message: Fix another DRC error and rotated battery JST connector
Parts:
- moved J2 2.02 mm to (55.0, 22.2), turned to 0 degrees
Routing:
- net BAT+: track 67.6 -> 66.2 mm
Changed lines of the file:
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@@
 	(footprint "Connector_JST:JST_PH_S2B-PH-K_1x02_P2.00mm_Horizontal"
 		(layer "F.Cu")
-		(at 54 24 90)
+		(at 55 22.25)
 		(descr "JST PH series connector, S2B-PH-K (http://www.jst-mfg.com/product/pdf/eng/ePH.pdf)")
 		(tags "connector JST PH horizontal")
 		(property "Reference" "J2"
-			(at 1 -2.55 90)
+			(at 1 -2.55 0)
 			(layer "F.SilkS")
 			(effects
@@
 		)
 		(property "Value" "Conn_01x02"
-			(at 1 7.45 90)
+			(at 1 7.45 0)
 			(layer "F.Fab")
 			(effects
@@
 		)
 		(property "Datasheet" ""
-			(at 0 0 90)
+			(at 0 0 0)
 			(layer "F.Fab")
 			(hide yes)
@@
 		)
 		(property "Description" "Generic connector, single row, 01x02, script generated (kicad-library-utils/schlib/autogen/connector/)"
-			(at 0 0 90)
+			(at 0 0 0)
 			(layer "F.Fab")
 			(hide yes)
@@
 		(duplicate_pad_numbers_are_jumpers no)
 		(fp_line
-			(start 4.06 -1.46)
-			(end 3.14 -1.46)
+			(start -2.06 -1.46)
+			(end -2.06 6.36)
 			(stroke
 				(width 0.12)
@@
 		)
 		(fp_line
-			(start 3.14 -1.46)
-			(end 3.14 0.14)
+			(start -2.06 0.14)
+			(end -1.14 0.14)
 			(stroke
 				(width 0.12)
@@
 		)
 		(fp_line
-			(start -1.14 -1.46)
-			(end -2.06 -1.46)
+			(start -2.06 6.36)
+			(end 4.06 6.36)
 			(stroke
 				(width 0.12)
@@
 		)
 		(fp_line
-			(start -2.06 -1.46)
-			(end -2.06 6.36)
+			(start -1.14 -1.46)
+			(end -2.06 -1.46)
 			(stroke
 				(width 0.12)
@@
 		)
 		(fp_line
-			(start 4.06 0.14)
-			(end 3.14 0.14)
+			(start -1.14 0.14)
+			(end -1.14 -1.46)
 			(stroke
 				(width 0.12)
@@
 		)
 		(fp_line
-			(start 3.14 0.14)
-			(end 2.86 0.14)
+			(start -0.86 0.14)
+			(end -1.14 0.14)
 			(stroke
 				(width 0.12)
@@
 		)
 		(fp_line
-			(start -0.86 0.14)
-			(end -1.14 0.14)
+			(start -0.8 4.1)
+			(end -0.8 6.36)
 			(stroke
 				(width 0.12)
@@
 		)
 		(fp_line
-			(start -1.14 0.14)
-			(end -1.14 -1.46)
+			(start -0.3 4.1)
+			(end -0.3 6.36)
 			(stroke
 				(width 0.12)
@@
 		)
 		(fp_line
-			(start -2.06 0.14)
-			(end -1.14 0.14)
+			(start 0.5 2)
+			(end 1.5 2)
 			(stroke
 				(width 0.12)
@@
 		)
 		(fp_line
-			(start 1.5 2)
-			(end 1.5 6.36)
+			(start 0.5 6.36)
+			(end 0.5 2)
 			(stroke
 				(width 0.12)
@@
 		)
 		(fp_line
-			(start 0.5 2)
-			(end 1.5 2)
+			(start 1.5 2)
+			(end 1.5 6.36)
 			(stroke
 				(width 0.12)
@@
 		)
 		(fp_line
-			(start -0.3 4.1)
-			(end -0.3 6.36)
+			(start 3.14 -1.46)
+			(end 3.14 0.14)
 			(stroke
 				(width 0.12)
@@
 		)
 		(fp_line
-			(start -0.8 4.1)
-			(end -0.8 6.36)
+			(start 3.14 0.14)
+			(end 2.86 0.14)
 			(stroke
 				(width 0.12)
@@
 		)
 		(fp_line
-			(start 4.06 6.36)
-			(end 4.06 -1.46)
+			(start 4.06 -1.46)
+			(end 3.14 -1.46)
 			(stroke
 				(width 0.12)
@@
 		)
 		(fp_line
-			(start 0.5 6.36)
-			(end 0.5 2)
+			(start 4.06 0.14)
+			(end 3.14 0.14)
 			(stroke
 				(width 0.12)
@@
 		)
 		(fp_line
-			(start -2.06 6.36)
-			(end 4.06 6.36)
+			(start 4.06 6.36)
+			(end 4.06 -1.46)
 			(stroke
 				(width 0.12)
@@
 		)
 		(fp_rect
-			(start 2.3 2.5)
-			(end 3.3 4.1)
+			(start -1.3 2.5)
+			(end -0.3 4.1)
 			(stroke
 				(width 0.12)
@@
 		)
 		(fp_rect
-			(start -1.3 2.5)
-			(end -0.3 4.1)
+			(start 2.3 2.5)
+			(end 3.3 4.1)
 			(stroke
 				(width 0.12)
@@
 		)
 		(fp_line
-			(start 3.95 -1.35)
-			(end 3.25 -1.35)
+			(start -1.95 -1.35)
+			(end -1.95 6.25)
 			(stroke
 				(width 0.1)
@@
 		)
 		(fp_line
-			(start 3.25 -1.35)
-			(end 3.25 0.25)
+			(start -1.95 6.25)
+			(end 3.95 6.25)
 			(stroke
 				(width 0.1)
@@
 		)
 		(fp_line
-			(start -1.95 -1.35)
-			(end -1.95 6.25)
+			(start -1.25 0.25)
+			(end -1.25 -1.35)
 			(stroke
 				(width 0.1)
@@
 		)
 		(fp_line
-			(start 3.25 0.25)
-			(end -1.25 0.25)
+			(start -0.5 1.375)
+			(end 0.5 1.375)
 			(stroke
 				(width 0.1)
@@
 		)
 		(fp_line
-			(start -1.25 0.25)
-			(end -1.25 -1.35)
+			(start 0 0.875)
+			(end -0.5 1.375)
 			(stroke
 				(width 0.1)
@@
 		)
 		(fp_line
-			(start 0 0.875)
-			(end -0.5 1.375)
+			(start 0.5 1.375)
+			(end 0 0.875)
 			(stroke
 				(width 0.1)
@@
 		)
 		(fp_line
-			(start 0.5 1.375)
-			(end 0 0.875)
+			(start 3.25 -1.35)
+			(end 3.25 0.25)
 			(stroke
 				(width 0.1)
@@
 		)
 		(fp_line
-			(start -0.5 1.375)
-			(end 0.5 1.375)
+			(start 3.25 0.25)
+			(end -1.25 0.25)
 			(stroke
 				(width 0.1)
@@
 		)
 		(fp_line
-			(start 3.95 6.25)
-			(end 3.95 -1.35)
+			(start 3.95 -1.35)
+			(end 3.25 -1.35)
 			(stroke
 				(width 0.1)
@@
 		)
 		(fp_line
-			(start -1.95 6.25)
-			(end 3.95 6.25)
+			(start 3.95 6.25)
+			(end 3.95 -1.35)
 			(stroke
 				(width 0.1)
@@
 		)
 		(fp_text user "${REFERENCE}"
-			(at 1 2.5 90)
+			(at 1 2.5 0)
 			(layer "F.Fab")
 			(effects
@@
 		)
 		(pad "1" thru_hole roundrect
-			(at 0 0 90)
+			(at 0 0)
 			(size 1.2 1.75)
 			(drill 0.75)
@@
 		)
 		(pad "2" thru_hole oval
-			(at 2 0 90)
+			(at 2 0)
 			(size 1.2 1.75)
 			(drill 0.75)
@@
 	)
 	(via
-		(at 46.5 20.25)
+		(at 46.5 21)
 		(size 0.6)
 		(drill 0.3)
@@
 	)
 	(segment
+		(start 55 20.775)
+		(end 51.5 17.275)
+		(width 0.5)
+		(layer "F.Cu")
+		(net "BAT+")
+	)
+	(segment
 		(start 52.8 14.196522)
 		(end 52.8 15.975)
@@
 	)
 	(segment
-		(start 51.5 21.5)
-		(end 54 24)
-		(width 0.5)
-		(layer "F.Cu")
-		(net "BAT+")
-	)
-	(segment
 		(start 32.202541 14.095)
 		(end 31.744113 13.636572)
@@
 	)
 	(segment
-		(start 51.5 17.275)
-		(end 51.5 21.5)
-		(width 0.5)
-		(layer "F.Cu")
-		(net "BAT+")
-	)
-	(segment
 		(start 33.525 14.095)
 		(end 32.202541 14.095)
@@
 		(width 0.5)
 		(layer "F.Cu")
+		(net "BAT+")
+	)
+	(segment
+		(start 55 22.25)
+		(end 55 20.775)
+		(width 0.5)
+		(layer "F.Cu")

Commit message: idk tbh
Parts:
- moved SW2 9.51 mm to (56.5, 43.5)
- moved C6 9.20 mm to (50.2, 44.5)
- moved R7 9.20 mm to (50.2, 41.2)
- moved C5 8.53 mm to (50.8, 48.5)
- moved SW1 8.53 mm to (56.8, 50.5)
- moved R6 8.50 mm to (50.2, 52.5)
Routing:
- net +3V3: track 89.7 -> 78.5 mm
- net EN: track 36.9 -> 41.1 mm
- net IO0: track 34.0 -> 38.0 mm
- net Net-(R6-Pad2): track 8.37 -> 8.87 mm
Changed lines of the file:
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@@
 	(footprint "Capacitor_SMD:C_0603_1608Metric"
 		(layer "F.Cu")
-		(at 50 40 180)
+		(at 50.75 48.5 180)
 		(descr "Capacitor SMD 0603 (1608 Metric), square (rectangular) end terminal, IPC-7351 nominal, (Body size source: IPC-SM-782 page 76, https://www.pcb-3d.com/wordpress/wp-content/uploads/ipc-sm-782a_amendment_1_and_2.pdf)")
 		(tags "capacitor")
@@
 	(footprint "Resistor_SMD:R_0603_1608Metric"
 		(layer "F.Cu")
-		(at 50 44)
+		(at 50.25 52.5)
 		(descr "Resistor SMD 0603 (1608 Metric), square (rectangular) end terminal, IPC-7351 nominal, (Body size source: IPC-SM-782 page 72, https://www.pcb-3d.com/wordpress/wp-content/uploads/ipc-sm-782a_amendment_1_and_2.pdf)")
 		(tags "resistor")
@@
 	(footprint "Capacitor_SMD:C_0603_1608Metric"
 		(layer "F.Cu")
-		(at 50 35.275 -90)
+		(at 50.25 44.475 -90)
 		(descr "Capacitor SMD 0603 (1608 Metric), square (rectangular) end terminal, IPC-7351 nominal, (Body size source: IPC-SM-782 page 76, https://www.pcb-3d.com/wordpress/wp-content/uploads/ipc-sm-782a_amendment_1_and_2.pdf)")
 		(tags "capacitor")
@@
 	(footprint "Button_Switch_SMD:SW_SPST_TL3342"
 		(layer "F.Cu")
-		(at 56 34)
+		(at 56.5 43.5)
 		(descr "Low-profile SMD Tactile Switch, https://www.e-switch.com/system/asset/product_line/data_sheet/165/TL3342.pdf")
 		(tags "SPST Tactile Switch")
@@
 	(footprint "Resistor_SMD:R_0603_1608Metric"
 		(layer "F.Cu")
-		(at 50 32 -90)
+		(at 50.25 41.2 -90)
 		(descr "Resistor SMD 0603 (1608 Metric), square (rectangular) end terminal, IPC-7351 nominal, (Body size source: IPC-SM-782 page 72, https://www.pcb-3d.com/wordpress/wp-content/uploads/ipc-sm-782a_amendment_1_and_2.pdf)")
 		(tags "resistor")
@@
 	(footprint "Button_Switch_SMD:SW_SPST_TL3342"
 		(layer "F.Cu")
-		(at 56 42 180)
+		(at 56.75 50.5 180)
 		(descr "Low-profile SMD Tactile Switch, https://www.e-switch.com/system/asset/product_line/data_sheet/165/TL3342.pdf")
 		(tags "SPST Tactile Switch")
@@
 	)
 	(segment
-		(start 59.15 40.1)
-		(end 52.85 40.1)
+		(start 53.5 48.5)
+		(end 53.6 48.6)
 		(width 0.25)
 		(layer "F.Cu")
@@
 	)
 	(segment
-		(start 52.85 40.1)
-		(end 50.875 40.1)
+		(start 51.525 48.5)
+		(end 53.5 48.5)
 		(width 0.25)
 		(layer "F.Cu")
@@
 	)
 	(segment
-		(start 50.875 40.1)
-		(end 50.775 40)
+		(start 53.6 48.6)
+		(end 59.9 48.6)
 		(width 0.25)
 		(layer "F.Cu")
@@
 	)
 	(segment
-		(start 45.8 34.87)
-		(end 49.495 31.175)
+		(start 44.435 41.34)
+		(end 42.5 43.275)
 		(width 0.5)
 		(layer "F.Cu")
@@
 	)
 	(segment
-		(start 44.435 41.34)
-		(end 42.5 43.275)
+		(start 50.25 40.375)
+		(end 47.625 40.375)
 		(width 0.5)
 		(layer "F.Cu")
@@
 	)
 	(segment
-		(start 37.9125 25)
-		(end 47 25)
-		(width 0.5)
-		(layer "F.Cu")
-		(net "+3V3")
-	)
-	(segment
 		(start 14.775 48)
 		(end 14.775 45.753358)
@@
 	)
 	(segment
-		(start 50 28)
-		(end 50 31.175)
-		(width 0.5)
-		(layer "F.Cu")
-		(net "+3V3")
-	)
-	(segment
 		(start 39 29.42)
 		(end 40.35 29.42)
@@
 	)
 	(segment
-		(start 34.8625 21.95)
-		(end 37.9125 25)
+		(start 33.175 21.95)
+		(end 33 21.775)
 		(width 0.5)
 		(layer "F.Cu")
@@
 	)
 	(segment
-		(start 33.175 21.95)
+		(start 31 21.775)
 		(end 33 21.775)
 		(width 0.5)
@@
 	)
 	(segment
-		(start 47 25)
-		(end 50 28)
+		(start 47.625 40.375)
+		(end 46.66 41.34)
 		(width 0.5)
 		(layer "F.Cu")
@@
 	)
 	(segment
-		(start 49.495 31.175)
-		(end 50 31.175)
+		(start 14.46 52.5)
+		(end 14.46 50.315)
 		(width 0.5)
 		(layer "F.Cu")
@@
 	)
 	(segment
-		(start 31 21.775)
-		(end 33 21.775)
+		(start 44.5 41.34)
+		(end 44.435 41.34)
 		(width 0.5)
 		(layer "F.Cu")
@@
 	)
 	(segment
-		(start 14.46 52.5)
-		(end 14.46 50.315)
+		(start 39 26.0875)
+		(end 39 29.42)
 		(width 0.5)
 		(layer "F.Cu")
@@
 	)
 	(segment
-		(start 44.5 41.34)
-		(end 44.435 41.34)
+		(start 34.8625 21.95)
+		(end 39 26.0875)
+		(width 0.5)
+		(layer "F.Cu")
+		(net "+3V3")
+	)
+	(segment
+		(start 46.66 41.34)
+		(end 44.5 41.34)
 		(width 0.5)
 		(layer "F.Cu")
@@
 	)
 	(segment
-		(start 44.013299 45.055)
-		(end 44.986701 45.055)
-		(width 0.25)
-		(layer "F.Cu")
-		(net "EN")
-	)
-	(segment
-		(start 33.9325 43.5675)
-		(end 34.365 44)
-		(width 0.25)
-		(layer "F.Cu")
-		(net "EN")
-	)
-	(segment
 		(start 22.558058 42.941942)
 		(end 22 43.5)
@@
 	)
 	(segment
-		(start 45.675 44)
-		(end 49.175 44)
-		(width 0.25)
-		(layer "F.Cu")
-		(net "EN")
-	)
-	(segment
-		(start 38.513299 43.485)
-		(end 39.486701 43.485)
+		(start 48.5 51.575)
+		(end 48.5 48.568299)
 		(width 0.25)
 		(layer "F.Cu")
@@
 	(segment
 		(start 34.365 44)
-		(end 37.998299 44)
-		(width 0.25)
-		(layer "F.Cu")
-		(net "EN")
-	)
-	(segment
-		(start 37.998299 44)
-		(end 38.513299 43.485)
+		(end 33.9325 43.5675)
 		(width 0.25)
 		(layer "F.Cu")
@@
 	)
 	(segment
-		(start 39.486701 43.485)
-		(end 40.001701 44)
+		(start 49.425 52.5)
+		(end 48.5 51.575)
 		(width 0.25)
 		(layer "F.Cu")
@@
 	)
 	(segment
-		(start 45.675 44.366701)
-		(end 45.675 44)
+		(start 41.056701 45.055)
+		(end 39.486701 43.485)
 		(width 0.25)
 		(layer "F.Cu")
@@
 	)
 	(segment
-		(start 43.325 44.366701)
-		(end 44.013299 45.055)
+		(start 37.998299 44)
+		(end 34.365 44)
 		(width 0.25)
 		(layer "F.Cu")
@@
 	)
 	(segment
-		(start 40.001701 44)
-		(end 43.325 44)
+		(start 48.5 48.568299)
+		(end 44.986701 45.055)
 		(width 0.25)
 		(layer "F.Cu")
@@
 	)
 	(segment
-		(start 43.325 44)
-		(end 43.325 44.366701)
+		(start 39.486701 43.485)
+		(end 38.513299 43.485)
 		(width 0.25)
 		(layer "F.Cu")
@@
 	)
 	(segment
-		(start 44.986701 45.055)
-		(end 45.675 44.366701)
+		(start 38.513299 43.485)
+		(end 37.998299 44)
 		(width 0.25)
 		(layer "F.Cu")
@@
 		(net "EN")
 	)
+	(segment
+		(start 44.986701 45.055)
+		(end 41.056701 45.055)
+		(width 0.25)
+		(layer "F.Cu")
+		(net "EN")
+	)
 	(via
 		(at 33.9325 43.5675)
@@
 	)
 	(segment
-		(start 50.825 44)
-		(end 52.75 44)
+		(start 59.9 52.4)
+		(end 53.6 52.4)
 		(width 0.25)
 		(layer "F.Cu")
@@
 	)
 	(segment
-		(start 52.85 43.9)
-		(end 59.15 43.9)
+		(start 53.5 52.5)
+		(end 53.6 52.4)
 		(width 0.25)
 		(layer "F.Cu")
@@
 	)
 	(segment
-		(start 52.75 44)
-		(end 52.85 43.9)
+		(start 51.075 52.5)
+		(end 53.5 52.5)
 		(width 0.25)
 		(layer "F.Cu")
@@
 	)
 	(segment
-		(start 59.15 32.1)
-		(end 52.85 32.1)
+		(start 48 41.5)
+		(end 49.725 41.5)
 		(width 0.25)
 		(layer "F.Cu")
@@
 	)
 	(segment
-		(start 50 32.825)
-		(end 50 34.5)
+		(start 50.275 42.025)
+		(end 50.7 41.6)
 		(width 0.25)
 		(layer "F.Cu")
@@
 	)
 	(segment
-		(start 49 34.5)
-		(end 48.5 34)
+		(start 50.7 41.6)
+		(end 53.35 41.6)
+		(width 0.25)
+		(layer "F.Cu")
+		(net "IO0")
+	)
+	(segment
+		(start 50.25 42.025)
+		(end 50.275 42.025)
 		(width 0.25)
 		(layer "F.Cu")
@@
 	)
 	(segment
-		(start 52.85 32.1)
-		(end 50.725 32.1)
+		(start 49.725 41.5)
+		(end 50.25 42.025)
 		(width 0.25)
 		(layer "F.Cu")
@@
 	)
 	(segment
-		(start 50 34.5)
-		(end 49 34.5)
+		(start 53.35 41.6)
+		(end 59.65 41.6)
 		(width 0.25)
 		(layer "F.Cu")
@@
 	)
 	(segment
-		(start 50.725 32.1)
-		(end 50 32.825)
+		(start 50.25 43.7)
+		(end 50.25 42.025)
 		(width 0.25)
 		(layer "F.Cu")
@@
 	)
 	(via
-		(at 48.5 34)
+		(at 48 41.5)
 		(size 0.6)
 		(drill 0.3)
@@
 	)
 	(segment
-		(start 39.411701 33.25)
+		(start 40.161701 34)
+		(end 39.411701 33.25)
+		(width 0.25)
+		(layer "B.Cu")
+		(net "IO0")
+	)
+	(segment
+		(start 40.5 34)
 		(end 40.161701 34)
 		(width 0.25)
@@
 	)
 	(segment
-		(start 31.5 28.5)
+		(start 36.25 33.25)
+		(end 31.5 28.5)
+		(width 0.25)
+		(layer "B.Cu")
+		(net "IO0")
+	)
+	(segment
+		(start 44.125 37.625)
+		(end 40.5 34)
+		(width 0.25)
+		(layer "B.Cu")
+		(net "IO0")
+	)
+	(segment
+		(start 48 41.5)
+		(end 45.675 39.175)
+		(width 0.25)
+		(layer "B.Cu")
+		(net "IO0")
+	)
+	(segment
+		(start 39.411701 33.25)
 		(end 36.25 33.25)
 		(width 0.25)
@@
 	)
 	(segment
-		(start 40.161701 34)
-		(end 48.5 34)
+		(start 44.986701 37.625)
+		(end 44.125 37.625)
 		(width 0.25)
 		(layer "B.Cu")
@@
 	)
 	(segment
-		(start 36.25 33.25)
-		(end 39.411701 33.25)
+		(start 45.675 38.313299)
+		(end 44.986701 37.625)
+		(width 0.25)
+		(layer "B.Cu")
+		(net "IO0")
+	)
+	(segment
+		(start 45.675 39.175)
+		(end 45.675 38.313299)
 		(width 0.25)
 		(layer "B.Cu")

Commit message: gerber and stuff
Parts:
- moved C10 8.40 mm to (46.8, 33.4), turned to 0 degrees
- moved C11 7.58 mm to (46.8, 31.2), turned to 0 degrees
Connections:
- C10 pad 1: Net-(C10-Pad1) -> BAT+
- C11 pad 2: Net-(C10-Pad1) -> GND
- C5 pad 1: Net-(C5-Pad1) -> EN
- J4 pad 5: +3V3 -> unconnected-(J4-Pin_5-Pad5)
- R6 pad 1: EN -> +3V3
- R6 pad 2: Net-(R6-Pad2) -> EN
- SW1 pad 1: Net-(R6-Pad2) -> EN
- SW1 pad 2: Net-(C5-Pad1) -> GND
Routing:
- net EN: track 41.1 -> 54.4 mm
- net +3V3: track 78.5 -> 90.9 mm, vias 1 -> 5
- net Net-(R6-Pad2): track 8.87 -> 0.00 mm
- net Net-(C5-Pad1): track 8.42 -> 0.00 mm
- net GND: track 16.5 -> 22.9 mm
- net Net-(C10-Pad1): track 1.67 -> 0.00 mm
- net BAT+: track 66.2 -> 64.9 mm, vias 3 -> 5
